File: pot_fleur/BQ25570.kicad_sch (KiCad schematic)
At the start: 29 parts, among them J10 P-MFC, J19 Conn_01x02_Socket, J5 Conn_01x02_Pin, J6 Conn_01x02_Pin, U3 BQ25570

Commit message: Update SmartPot schematic and BQ25570 configuration
Parts:
- LBOOST1: footprint LPS4018-223MRC:IND_LPS4018-223MRC -> LBOOST:IND_LPS4018-223MRC
Connections:
- no-connect marks 0 -> 3
Other:
- note added: "Deuxieme zone : Supercapa (on veut juste l empreinte)"
- note added: "EN : Pour le controler (utilisateur)"
- note added: "Pin mesure courant"
- note added: "Premiere zone : Supercapa (on veut juste l empreinte)"
- note added: "on veut juste les empreintes ici car on va regler la tension capa, cycle hyteris"
- note added: "super condo 10F"
Changed lines of the file:
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@@
 	(generator_version "10.0")
 	(paper "A4")
+	(text "on veut juste les empreintes ici \ncar on va regler la tension capa, cycle hyteris\n"
+		(exclude_from_sim no)
+		(at 241.808 124.46 0)
+		(effects
+			(font
+				(size 1.27 1.27)
+			)
+		)
+	)
+	(text "Premiere zone : \nSupercapa (on veut juste l empreinte)"
+		(exclude_from_sim no)
+		(at 166.37 19.558 0)
+		(effects
+			(font
+				(size 1.27 1.27)
+			)
+		)
+	)
+	(text "super condo 10F "
+		(exclude_from_sim no)
+		(at 167.64 24.638 0)
+		(effects
+			(font
+				(size 1.27 1.27)
+			)
+		)
+	)
+	(text "Deuxieme zone : \nSupercapa (on veut juste l empreinte)\n"
+		(exclude_from_sim no)
+		(at 96.52 94.996 0)
+		(effects
+			(font
+				(size 1.27 1.27)
+			)
+		)
+	)
+	(text "EN : \nPour le controler (utilisateur)"
+		(exclude_from_sim no)
+		(at 120.904 72.644 0)
+		(effects
+			(font
+				(size 1.27 1.27)
+			)
+		)
+	)
+	(text "Pin mesure courant\n"
+		(exclude_from_sim no)
+		(at 40.64 77.216 0)
+		(effects
+			(font
+				(size 1.27 1.27)
+			)
+		)
+	)
 	(junction
 		(at 184.15 95.25)
@@
 		(diameter 0)
 		(color 0 0 0 0)
+	)
+	(no_connect
+		(at 148.59 72.39)
+	)
+	(no_connect
+		(at 147.32 81.28)
+	)
+	(no_connect
+		(at 119.38 76.2)
 	)
 	(wire
@@
 			)
 		)
-		(property "Footprint" "LPS4018-223MRC:IND_LPS4018-223MRC"
+		(property "Footprint" "LBOOST:IND_LPS4018-223MRC"
 			(at 133.35 63.5 0)
 			(hide yes)

Commit message: Add preliminary four-layer routing and 868 MHz PCB antenna
Parts:
- ROK1: value 4.22M -> 4.12M
- ROK3: value 1.1M -> 1.02M
Changed lines of the file:
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@@
 			)
 		)
-		(property "Value" "1.1M"
+		(property "Value" "1.02M"
 			(at 219.71 93.9799 0)
 			(show_name no)
@@
 			)
 		)
-		(property "Value" "4.22M"
+		(property "Value" "4.12M"
 			(at 219.71 118.1099 0)
 			(show_name no)
