File: pot_fleur/capteur.kicad_sch (KiCad schematic)
At the start: 12 parts, among them J7 Conn_01x03_Pin, Q1 Q_PMOS_GSD, U2 BME280, U4 SHT40-AD1B-R2

Commit message: Update SmartPot schematic and BQ25570 configuration
Parts:
- removed C1, C2: 100nF, symbol Device:C
- removed J7: Conn_01x03_Pin, SHT40-AD1B-R2:SHT4X, symbol Connector:Conn_01x03_Pin
- removed Q1: Q_PMOS_GSD, Package_QFP:TQFP-44_10x10mm_P0.8mm, symbol Transistor_FET:Q_PMOS_GSD
- removed R1, R2: 4,7k, symbol Device:R
- removed R10: 100k, symbol Device:R
- removed U2: BME280, Package_LGA:Bosch_LGA-8_2.5x2.5mm_P0.65mm_ClockwisePinNumbering, symbol Sensor:BME280
- added J7: Conn_01x04_Pin, Connector_PinHeader_2.54mm:PinHeader_1x02_P2.54mm_Vertical, symbol Connector:Conn_01x04_Pin
- C5: footprint SHT40-AD1B-R2:SHT4X -> Capacitor_SMD:C_0603_1608Metric
- R8, R9: footprint (none) -> Resistor_SMD:R_0603_1608Metric
- U4: footprint SHT40-AD1B-R2:SHT4X -> SHT40:SHT4X
Connections:
- net GND: now also J7.4 (Pin_4)
- net PWR: now also J7.1 (Pin_1)
- new net SOIL_SCL: J7.3 (Pin_3)
- new net SOIL_SDA: J7.2 (Pin_2)
Other:
- note added: "Capteur Adafruit STEMMA Soil Sensor #4026 Humi Terre"
- note removed: "Alimentation MOS P-Channel : DMP2305U vers capteur EC-5"
- note removed: "Capteur BME280 Humi, Press, Temp"
- note removed: "Capteur EC-5 Humi Terre"
- note removed: "D"
- note removed: "G"
- note removed: "S"

Commit message: Add preliminary four-layer routing and 868 MHz PCB antenna
Parts:
- J7: footprint Connector_PinHeader_2.54mm:PinHeader_1x02_P2.54mm_Vertical -> Connector_PinHeader_2.54mm:PinHeader_1x04_P2.54mm_Vertical
Changed lines of the file:
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@@
 			)
 		)
-		(property "Footprint" "Connector_PinHeader_2.54mm:PinHeader_1x02_P2.54mm_Vertical"
+		(property "Footprint" "Connector_PinHeader_2.54mm:PinHeader_1x04_P2.54mm_Vertical"
 			(at 219.71 100.33 0)
 			(hide yes)
