File: pot_fleur/pot_fleur.kicad_pcb (KiCad board)
At the start: 4 copper layers, 30 x 60 mm, 48 parts, among them J1 Conn_01x04_Pin, J10 P-MFC, J19 Conn_01x02_Socket, J2 Conn_01x04_Pin, J3 Conn_Coaxial_Small, J4 Conn_01x04_Pin, J5 Conn_01x02_Pin, J6 Conn_01x02_Pin, J7 Conn_01x04_Pin, SW1 B3U-1000P, SW2 B3U-1000P, U1 RAK3172-xx-8-SM-xI, U3 BQ25570, U4 SHT40-AD1B-R2

Commit message: Use required 0603 packages for antenna matching network
Parts:
- C6, C7: footprint Capacitor_SMD:C_0402_1005Metric -> Capacitor_SMD:C_0603_1608Metric
- L1: footprint Inductor_SMD:L_0402_1005Metric -> Inductor_SMD:L_0603_1608Metric
- moved R4 1.26 mm to (62.0, 67.8)
- moved C6 1.10 mm to (59.6, 69.0)
- moved L1 0.81 mm to (57.3, 67.7)
Routing:
- net GND: track 193.0 -> 185.6 mm, vias 5 -> 4
- net /Microcontroleur/RF_FEED: track 8.86 -> 10.1 mm
- net Net-(J3-In): track 30.5 -> 31.5 mm

Commit message: Replace TI radiator with adapted CST SmartPot IFA antenna
Parts:
- removed C7: 1pF, Capacitor_SMD:C_0603_1608Metric
- added R6: 0, Resistor_SMD:R_0603_1608Metric, F.Cu at (52.0, 63.5)
- A1: value PCB_868MHz_TI_DN038 -> PCB_868MHz_CST_IFA; footprint SmartPot_RF:TI_DN038_868MHz_Helical -> SmartPot_RF:CST_IFA_868MHz_SmartPot
- L1: value 12nH -> DNP
- moved C6 6.18 mm to (54.2, 66.0)
- moved A1 5.77 mm to (52.0, 61.0)
- moved R4 5.49 mm to (57.2, 65.2)
- moved L1 5.13 mm to (54.4, 63.5)
Routing:
- net GND: track 185.6 -> 179.2 mm, vias 4 -> 3
- net /Microcontroleur/RF_FEED: track 10.1 -> 14.8 mm
- net Net-(J3-In): track 31.5 -> 34.8 mm
