File: pot_fleur/untitled.kicad_sch (KiCad schematic)
At the start: 14 parts, among them J1 Conn_01x04_Pin, J2 Conn_01x04_Pin, J3 Conn_Coaxial_Small, J4 Conn_01x04_Pin, SW1 SW_DPST_x2, SW2 SW_DPST_x2, U1 RAK3172-xx-8-SM-xI

Commit message: Update SmartPot schematic and BQ25570 configuration
Parts:
- C3: footprint (none) -> Capacitor_SMD:C_0603_1608Metric
- J1, J2, J4: footprint (none) -> Connector_PinHeader_2.54mm:PinHeader_1x02_P2.54mm_Vertical
- R3, R4, R5, R6, R7, SW1: footprint (none) -> Resistor_SMD:R_0603_1608Metric
Other:
- note removed: "EC-5 RAK3172 SOIL_OUT ──────────────────► PB2 / PIN_A2 pin module 26 SOIL_EN ──────────────────► PA0 pin module 29"
Changed lines of the file:
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@@
-		)
-	)
-	(text "EC-5                         RAK3172\n\nSOIL_OUT ──────────────────► PB2 / PIN_A2\n                              pin module 26\n\nSOIL_EN  ──────────────────► PA0\n                              pin module 29"
-		(exclude_from_sim no)
-		(at 137.922 141.986 0)
-		(effects
-			(font
-				(size 1.27 1.27)
-			)
 		)
 	)
@@
 	(wire
 		(pts
-			(xy 91.44 60.96) (xy 116.84 60.96)
-		)
-		(stroke
-			(width 0)
-			(type default)
-		)
-	)
-	(wire
-		(pts
-			(xy 168.91 91.44) (xy 157.48 91.44)
+			(xy 157.48 91.44) (xy 184.15 91.44)
 		)
 		(stroke
@@
 	(wire
 		(pts
+			(xy 157.48 60.96) (xy 168.91 60.96)
+		)
+		(stroke
+			(width 0)
+			(type default)
+		)
+	)
+	(wire
+		(pts
 			(xy 191.77 53.34) (xy 198.12 53.34)
 		)
@@
 	(wire
 		(pts
-			(xy 168.91 88.9) (xy 157.48 88.9)
+			(xy 157.48 88.9) (xy 184.15 88.9)
 		)
 		(stroke
@@
 	(wire
 		(pts
-			(xy 157.48 60.96) (xy 177.8 60.96)
-		)
-		(stroke
-			(width 0)
-			(type default)
-		)
-	)
-	(wire
-		(pts
 			(xy 259.08 116.84) (xy 251.46 116.84)
 		)
@@
 		(pts
 			(xy 171.45 53.34) (xy 168.91 53.34)
+		)
+		(stroke
+			(width 0)
+			(type default)
+		)
+	)
+	(wire
+		(pts
+			(xy 107.95 60.96) (xy 116.84 60.96)
 		)
 		(stroke
@@
 		)
 	)
-	(global_label "SOIL_OUT"
-		(shape input)
-		(at 91.44 60.96 180)
-		(fields_autoplaced yes)
-		(effects
-			(font
-				(size 1.27 1.27)
-			)
-			(justify right)
-		)
-		(property "Intersheetrefs" "${INTERSHEET_REFS}"
-			(at 79.6857 60.96 0)
-			(hide yes)
-			(show_name no)
-			(do_not_autoplace no)
-			(effects
-				(font
-					(size 1.27 1.27)
-				)
-				(justify right)
-			)
-		)
-	)
 	(global_label "BOOT"
 		(shape input)
@@
 		)
 	)
+	(global_label "SOIL_SDA"
+		(shape bidirectional)
+		(at 184.15 88.9 0)
+		(fields_autoplaced yes)
+		(effects
+			(font
+				(size 1.27 1.27)
+			)
+			(justify left)
+		)
+		(property "Intersheetrefs" "${INTERSHEET_REFS}"
+			(at 196.9551 88.9 0)
+			(hide yes)
+			(show_name no)
+			(do_not_autoplace no)
+			(effects
+				(font
+					(size 1.27 1.27)
+				)
+				(justify left)
+			)
+		)
+	)
 	(global_label "PA8"
 		(shape bidirectional)
@@
 		)
 	)
+	(global_label "SOIL_SCL"
+		(shape bidirectional)
+		(at 184.15 91.44 0)
+		(fields_autoplaced yes)
+		(effects
+			(font
+				(size 1.27 1.27)
+			)
+			(justify left)
+		)
+		(property "Intersheetrefs" "${INTERSHEET_REFS}"
+			(at 196.8946 91.44 0)
+			(hide yes)
+			(show_name no)
+			(do_not_autoplace no)
+			(effects
+				(font
+					(size 1.27 1.27)
+				)
+				(justify left)
+			)
+		)
+	)
 	(global_label "PWR"
 		(shape input)
@@
 		(property "Intersheetrefs" "${INTERSHEET_REFS}"
 			(at 271.3785 36.83 0)
-			(hide yes)
-			(show_name no)
-			(do_not_autoplace no)
-			(effects
-				(font
-					(size 1.27 1.27)
-				)
-				(justify left)
-			)
-		)
-	)
-	(global_label "SOIL_EN"
-		(shape input)
-		(at 177.8 60.96 0)
-		(fields_autoplaced yes)
-		(effects
-			(font
-				(size 1.27 1.27)
-			)
-			(justify left)
-		)
-		(property "Intersheetrefs" "${INTERSHEET_REFS}"
-			(at 188.4052 60.96 0)
 			(hide yes)
 			(show_name no)
@@
 			)
 		)
-		(property "Footprint" ""
+		(property "Footprint" "Resistor_SMD:R_0603_1608Metric"
 			(at 189.992 59.69 90)
 			(hide yes)
@@
 			)
 		)
-		(property "Footprint" ""
+		(property "Footprint" "Resistor_SMD:R_0603_1608Metric"
 			(at 202.692 59.69 90)
 			(hide yes)
@@
 			)
 		)
-		(property "Footprint" ""
+		(property "Footprint" "Capacitor_SMD:C_0603_1608Metric"
 			(at 247.3452 95.25 0)
 			(hide yes)
@@
 			)
 		)
-		(property "Footprint" ""
+		(property "Footprint" "Resistor_SMD:R_0603_1608Metric"
 			(at 252.73 60.96 0)
 			(hide yes)
@@
 			)
 		)
-		(property "Footprint" ""
+		(property "Footprint" "Resistor_SMD:R_0603_1608Metric"
 			(at 165.1 55.118 90)
 			(hide yes)
@@
 			)
 		)
-		(property "Footprint" ""
+		(property "Footprint" "Connector_PinHeader_2.54mm:PinHeader_1x02_P2.54mm_Vertical"
 			(at 246.38 116.84 0)
 			(hide yes)
@@
 			)
 		)
-		(property "Footprint" ""
+		(property "Footprint" "Connector_PinHeader_2.54mm:PinHeader_1x02_P2.54mm_Vertical"
 			(at 243.84 36.83 0)
 			(hide yes)
@@
 			)
 		)
-		(property "Footprint" ""
+		(property "Footprint" "Connector_PinHeader_2.54mm:PinHeader_1x02_P2.54mm_Vertical"
 			(at 247.65 140.97 0)
 			(hide yes)
@@
 			)
 		)
-		(property "Footprint" ""
+		(property "Footprint" "Resistor_SMD:R_0603_1608Metric"
 			(at 198.12 66.548 90)
 			(hide yes)
@@
 			)
 		)
-		(property "Footprint" ""
+		(property "Footprint" "Resistor_SMD:R_0603_1608Metric"
 			(at 245.872 64.77 90)
 			(hide yes)

Commit message: Add preliminary four-layer routing and 868 MHz PCB antenna
Parts:
- A1: value (none) -> PCB_868MHz_TI_DN038; footprint (none) -> SmartPot_RF:TI_DN038_868MHz_Helical; now left out of the parts list
- C6: renamed from R5; value R -> DNP; footprint Resistor_SMD:R_0603_1608Metric -> Capacitor_SMD:C_0402_1005Metric; symbol Device:R -> Device:C; now not fitted
- C7: renamed from R6; value 0 -> 1pF; footprint Resistor_SMD:R_0603_1608Metric -> Capacitor_SMD:C_0402_1005Metric; symbol Device:R -> Device:C
- J1, J2, J4: footprint Connector_PinHeader_2.54mm:PinHeader_1x02_P2.54mm_Vertical -> Connector_PinHeader_2.54mm:PinHeader_1x04_P2.54mm_Vertical
- J3: footprint Package_DFN_QFN:WDFN-10-1EP_3x3mm_P0.5mm_EP1.8x2.5mm -> Connector_Coaxial:U.FL_Hirose_U.FL-R-SMT-1_Vertical; now not fitted
- L1: renamed from R7; value R -> 12nH; footprint Resistor_SMD:R_0603_1608Metric -> Inductor_SMD:L_0402_1005Metric; symbol Device:R -> Device:L
- R4: now not fitted
- SW1: value SW_DPST_x2 -> B3U-1000P; footprint Resistor_SMD:R_0603_1608Metric -> Button_Switch_SMD:SW_SPST_B3U-1000P; symbol Switch:SW_DPST_x2 -> Switch:SW_SPST
- SW2: value SW_DPST_x2 -> B3U-1000P; footprint Button_Switch_SMD:Nidec_Copal_CAS-120A -> Button_Switch_SMD:SW_SPST_B3U-1000P; symbol Switch:SW_DPST_x2 -> Switch:SW_SPST
Connections:
- net RF_FEED: now reaches C6.2, C7.1
- net RF_FEED: now also R4.1, U1.12 (RF)
Changed lines of the file:
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@@
 	)
 	(symbol
-		(lib_id "Device:R")
+		(lib_id "Device:C")
 		(at 191.77 59.69 0)
 		(unit 1)
@@
 		(on_board yes)
 		(in_pos_files yes)
-		(dnp no)
-		(fields_autoplaced yes)
-		(property "Reference" "R5"
+		(dnp yes)
+		(fields_autoplaced yes)
+		(property "Reference" "C6"
 			(at 194.31 58.4199 0)
 			(show_name no)
@@
 			)
 		)
-		(property "Value" "R"
+		(property "Value" "DNP"
 			(at 194.31 60.9599 0)
 			(show_name no)
@@
 			)
 		)
-		(property "Footprint" "Resistor_SMD:R_0603_1608Metric"
+		(property "Footprint" "Capacitor_SMD:C_0402_1005Metric"
 			(at 189.992 59.69 90)
 			(hide yes)
@@
 			(project "pot_fleur"
 				(path "/523f6adf-746e-4f97-9f6d-33bb6d5a221f/b9354401-9acc-46da-89c3-050c4bff531e"
-					(reference "R5")
-					(unit 1)
-				)
-			)
-		)
-	)
-	(symbol
-		(lib_id "Device:R")
+					(reference "C6")
+					(unit 1)
+				)
+			)
+		)
+	)
+	(symbol
+		(lib_id "Device:L")
 		(at 204.47 59.69 0)
 		(unit 1)
@@
 		(dnp no)
 		(fields_autoplaced yes)
-		(property "Reference" "R7"
+		(property "Reference" "L1"
 			(at 207.01 58.4199 0)
 			(show_name no)
@@
 			)
 		)
-		(property "Value" "R"
+		(property "Value" "12nH"
 			(at 207.01 60.9599 0)
 			(show_name no)
@@
 			)
 		)
-		(property "Footprint" "Resistor_SMD:R_0603_1608Metric"
+		(property "Footprint" "Inductor_SMD:L_0402_1005Metric"
 			(at 202.692 59.69 90)
 			(hide yes)
@@
 			(project "pot_fleur"
 				(path "/523f6adf-746e-4f97-9f6d-33bb6d5a221f/b9354401-9acc-46da-89c3-050c4bff531e"
-					(reference "R7")
+					(reference "L1")
 					(unit 1)
 				)
@@
 	)
 	(symbol
-		(lib_id "Switch:SW_DPST_x2")
+		(lib_id "Switch:SW_SPST")
 		(at 252.73 60.96 0)
 		(unit 1)
@@
 			)
 		)
-		(property "Value" "SW_DPST_x2"
+		(property "Value" "B3U-1000P"
 			(at 252.73 57.15 0)
 			(show_name no)
@@
 			)
 		)
-		(property "Footprint" "Resistor_SMD:R_0603_1608Metric"
+		(property "Footprint" "Button_Switch_SMD:SW_SPST_B3U-1000P"
 			(at 252.73 60.96 0)
 			(hide yes)
@@
 		(on_board yes)
 		(in_pos_files yes)
-		(dnp no)
+		(dnp yes)
 		(fields_autoplaced yes)
 		(property "Reference" "R4"
@@
 		(body_style 1)
 		(exclude_from_sim no)
-		(in_bom yes)
-		(on_board yes)
-		(in_pos_files yes)
+		(in_bom no)
+		(on_board yes)
+		(in_pos_files no)
 		(dnp no)
 		(fields_autoplaced yes)
@@
 			)
 		)
-		(property "Value" ""
+		(property "Value" "PCB_868MHz_TI_DN038"
 			(at 207.01 71.12 0)
 			(show_name no)
@@
 			)
 		)
-		(property "Footprint" ""
+		(property "Footprint" "SmartPot_RF:TI_DN038_868MHz_Helical"
 			(at 207.01 71.12 0)
 			(hide yes)
@@
 			)
 		)
-		(property "Datasheet" ""
+		(property "Datasheet" "https://www.ti.com/lit/an/swra416/swra416.pdf"
 			(at 207.01 71.12 0)
 			(hide yes)
@@
 			)
 		)
-		(property "Description" ""
+		(property "Description" "Printed helical radiator; pin 2 is ground reference, not radiator short"
 			(at 207.01 71.12 0)
 			(hide yes)
@@
 			)
 		)
-		(property "Footprint" "Connector_PinHeader_2.54mm:PinHeader_1x02_P2.54mm_Vertical"
+		(property "Footprint" "Connector_PinHeader_2.54mm:PinHeader_1x04_P2.54mm_Vertical"
 			(at 246.38 116.84 0)
 			(hide yes)
@@
 			)
 		)
-		(property "Footprint" "Connector_PinHeader_2.54mm:PinHeader_1x02_P2.54mm_Vertical"
+		(property "Footprint" "Connector_PinHeader_2.54mm:PinHeader_1x04_P2.54mm_Vertical"
 			(at 243.84 36.83 0)
 			(hide yes)
@@
 	)
 	(symbol
-		(lib_id "Switch:SW_DPST_x2")
+		(lib_id "Switch:SW_SPST")
 		(at 251.46 87.63 0)
 		(unit 1)
@@
 			)
 		)
-		(property "Value" "SW_DPST_x2"
+		(property "Value" "B3U-1000P"
 			(at 251.46 83.82 0)
 			(show_name no)
@@
 			)
 		)
-		(property "Footprint" "Button_Switch_SMD:Nidec_Copal_CAS-120A"
+		(property "Footprint" "Button_Switch_SMD:SW_SPST_B3U-1000P"
 			(at 251.46 87.63 0)
 			(hide yes)
@@
 		(on_board yes)
 		(in_pos_files yes)
-		(dnp no)
+		(dnp yes)
 		(fields_autoplaced yes)
 		(property "Reference" "J3"
@@
 			)
 		)
-		(property "Footprint" "Package_DFN_QFN:WDFN-10-1EP_3x3mm_P0.5mm_EP1.8x2.5mm"
+		(property "Footprint" "Connector_Coaxial:U.FL_Hirose_U.FL-R-SMT-1_Vertical"
 			(at 173.99 53.34 0)
 			(hide yes)
@@
 			)
 		)
-		(property "Footprint" "Connector_PinHeader_2.54mm:PinHeader_1x02_P2.54mm_Vertical"
+		(property "Footprint" "Connector_PinHeader_2.54mm:PinHeader_1x04_P2.54mm_Vertical"
 			(at 247.65 140.97 0)
 			(hide yes)
@@
 	)
 	(symbol
-		(lib_id "Device:R")
+		(lib_id "Device:C")
 		(at 198.12 64.77 90)
 		(unit 1)
@@
 		(dnp no)
 		(fields_autoplaced yes)
-		(property "Reference" "R6"
+		(property "Reference" "C7"
 			(at 198.12 58.42 90)
 			(show_name no)
@@
 			)
 		)
-		(property "Value" "0"
+		(property "Value" "1pF"
 			(at 198.12 60.96 90)
 			(show_name no)
@@
 			)
 		)
-		(property "Footprint" "Resistor_SMD:R_0603_1608Metric"
+		(property "Footprint" "Capacitor_SMD:C_0402_1005Metric"
 			(at 198.12 66.548 90)
 			(hide yes)
@@
 			(project "pot_fleur"
 				(path "/523f6adf-746e-4f97-9f6d-33bb6d5a221f/b9354401-9acc-46da-89c3-050c4bff531e"
-					(reference "R6")
+					(reference "C7")
 					(unit 1)
 				)
@@
 		)
 	)
+ (label "RF_FEED" (at 157.48 53.34 0) (effects (font (size 1.0 1.0)) (justify left bottom)))
+ (label "RF_FEED" (at 191.77 64.77 0) (effects (font (size 1.0 1.0)) (justify left bottom)))
 )

Commit message: Use required 0603 packages for antenna matching network
Parts:
- C6, C7: footprint Capacitor_SMD:C_0402_1005Metric -> Capacitor_SMD:C_0603_1608Metric
- L1: footprint Inductor_SMD:L_0402_1005Metric -> Inductor_SMD:L_0603_1608Metric
Changed lines of the file:
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@@
 			)
 		)
-		(property "Footprint" "Capacitor_SMD:C_0402_1005Metric"
+		(property "Footprint" "Capacitor_SMD:C_0603_1608Metric"
 			(at 189.992 59.69 90)
 			(hide yes)
@@
 			)
 		)
-		(property "Footprint" "Inductor_SMD:L_0402_1005Metric"
+		(property "Footprint" "Inductor_SMD:L_0603_1608Metric"
 			(at 202.692 59.69 90)
 			(hide yes)
@@
 			)
 		)
-		(property "Footprint" "Capacitor_SMD:C_0402_1005Metric"
+		(property "Footprint" "Capacitor_SMD:C_0603_1608Metric"
 			(at 198.12 66.548 90)
 			(hide yes)

Commit message: Replace TI radiator with adapted CST SmartPot IFA antenna
Parts:
- A1: value PCB_868MHz_TI_DN038 -> PCB_868MHz_CST_IFA; footprint SmartPot_RF:TI_DN038_868MHz_Helical -> SmartPot_RF:CST_IFA_868MHz_SmartPot
- L1: value 12nH -> DNP; now not fitted
- R6: renamed from C7; value 1pF -> 0; footprint Capacitor_SMD:C_0603_1608Metric -> Resistor_SMD:R_0603_1608Metric; symbol Device:C -> Device:R
Changed lines of the file:
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@@
 		(on_board yes)
 		(in_pos_files yes)
-		(dnp no)
+		(dnp yes)
 		(fields_autoplaced yes)
 		(property "Reference" "L1"
@@
 			)
 		)
-		(property "Value" "12nH"
+		(property "Value" "DNP"
 			(at 207.01 60.9599 0)
 			(show_name no)
@@
 			)
 		)
-		(property "Value" "PCB_868MHz_TI_DN038"
+		(property "Value" "PCB_868MHz_CST_IFA"
 			(at 207.01 71.12 0)
 			(show_name no)
@@
 			)
 		)
-		(property "Footprint" "SmartPot_RF:TI_DN038_868MHz_Helical"
+		(property "Footprint" "SmartPot_RF:CST_IFA_868MHz_SmartPot"
 			(at 207.01 71.12 0)
 			(hide yes)
@@
 			)
 		)
-		(property "Datasheet" "https://www.ti.com/lit/an/swra416/swra416.pdf"
+		(property "Datasheet" "https://github.com/MaxBarbe/SmartPot_RAK3172/blob/main/CST/TP1_M2_Smart_2-3.cst"
 			(at 207.01 71.12 0)
 			(hide yes)
@@
 			)
 		)
-		(property "Description" "Printed helical radiator; pin 2 is ground reference, not radiator short"
+		(property "Description" "CST IFA radiator; intentional short to GND through net tie; physical feed added, resimulation required"
 			(at 207.01 71.12 0)
 			(hide yes)
@@
 	)
 	(symbol
-		(lib_id "Device:C")
+		(lib_id "Device:R")
 		(at 198.12 64.77 90)
 		(unit 1)
@@
 		(dnp no)
 		(fields_autoplaced yes)
-		(property "Reference" "C7"
+		(property "Reference" "R6"
 			(at 198.12 58.42 90)
 			(show_name no)
@@
 			)
 		)
-		(property "Value" "1pF"
+		(property "Value" "0"
 			(at 198.12 60.96 90)
 			(show_name no)
@@
 			)
 		)
-		(property "Footprint" "Capacitor_SMD:C_0603_1608Metric"
+		(property "Footprint" "Resistor_SMD:R_0603_1608Metric"
 			(at 198.12 66.548 90)
 			(hide yes)
@@
 			(project "pot_fleur"
 				(path "/523f6adf-746e-4f97-9f6d-33bb6d5a221f/b9354401-9acc-46da-89c3-050c4bff531e"
-					(reference "C7")
-					(unit 1)
-				)
+					(reference "R6")
+					(unit 1)
+				)
