File: pot_fleur_v2_2couches/BQ25570.kicad_sch (KiCad schematic)
At the start: 29 parts, among them J10 P-MFC, J19 Conn_01x02_Socket, J5 Conn_01x02_Pin, J6 Conn_01x02_Pin, U3 BQ25570

Commit message: Adapt V2 energy input for soldered wires and add mask exports
Parts:
- J10: footprint TerminalBlock_Phoenix:TerminalBlock_Phoenix_MKDS-3-2-5.08_1x02_P5.08mm_Horizontal -> SmartPot_RF:Wire_Solder_2x_P5.08mm_D1.3mm; now left out of the parts list
Changed lines of the file:
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@@
 		(body_style 1)
 		(exclude_from_sim no)
-		(in_bom yes)
+		(in_bom no)
 		(on_board yes)
-		(in_pos_files yes)
+		(in_pos_files no)
 		(dnp no)
 		(property "Reference" "J10"
@@
 			)
 		)
-		(property "Footprint" "TerminalBlock_Phoenix:TerminalBlock_Phoenix_MKDS-3-2-5.08_1x02_P5.08mm_Horizontal"
+		(property "Footprint" "SmartPot_RF:Wire_Solder_2x_P5.08mm_D1.3mm"
 			(at 33.02 66.04 0)
 			(hide yes)
