File: pot_fleur_v2_2couches/pot_fleur.kicad_pcb (KiCad board)
At the start: 2 copper layers, 30 x 60 mm, 50 parts, among them J1 Conn_01x04_Pin, J10 P-MFC, J19 Conn_01x02_Socket, J2 Conn_01x04_Pin, J3 Conn_Coaxial_Small, J4 Conn_01x04_Pin, J5 Conn_01x02_Pin, J6 Conn_01x02_Pin, J7 Conn_01x04_Pin, SW1 B3U-1000P, SW2 B3U-1000P, U1 RAK3172-xx-8-SM-xI, U3 BQ25570, U4 SHT40-AD1B-R2

Commit message: Adapt V2 energy input for soldered wires and add mask exports
Parts:
- J10: footprint TerminalBlock_Phoenix:TerminalBlock_Phoenix_MKDS-3-2-5.08_1x02_P5.08mm_Horizontal -> SmartPot_RF:Wire_Solder_2x_P5.08mm_D1.3mm
